Commit message: Made assignments 1, 2,  and 3 mostly work

File: src/wasp_autonomous_systems/urdf/car.urdf (robot description, URDF)
Before this commit: robot car, 1 links, 0 joints
Links:
- link base_link: geometry visual mesh filename=package://wasp_autonomous_systems/meshes/car/car.dae scale=1.0 1.0 1.0
